File: HARDWARE/Temperature_Tire_Sensor/Temperature_Tire_Sensor.kicad_pcb (KiCad board)
At the start: 4 copper layers, 58 x 24 mm, 55 parts, among them IC1 MLX90621ESF-BAB-000-SP, J1 SWD_01x06, J2 CAN_01x04, SW1 RESET, U1 STM32L4P5RET6, U2 MIC5236, U3 MIC5306-2.6YD5-TR, U4 SN65HVD232, Y1 16MGHz

Commit message: merge
Parts:
- moved D2 0.50 mm to (110.2, 100.0)
Routing:
- net GND: track 53.7 -> 58.3 mm, vias 32 -> 41
- net /LED_OK: track 17.8 -> 16.3 mm
- net /CAN_L: track 21.3 -> 19.8 mm
- net /NRST: track 36.6 -> 37.8 mm
- net /CAN_H: track 19.6 -> 20.1 mm
- net /SWCLK: vias 0 -> 1
- added copper zone on B.Cu, net GND
- added copper zone on F.Cu, net GND
Other:
- board text added: "MATEUSZ KOZA"
- board text added: "TIRE TEMPERATURE SENSOR V1.0"
- board text removed: "Mateusz Koza"
- board text removed: "TTS V1.0"
